File: CtrlTree_hw/CtrlTree.sch (KiCad schematic (older format))
At the start: 150 parts, among them Q1 IRLML6401, Q2 IRLML0030, U1 USBLC6

Commit message: Layout started
Parts:
- removed C32: 10n, Capacitors:CAP_0603_Silks, symbol Tittar_kl:C
- removed HOLE1, HOLE2, HOLE3, HOLE4: HOLE_METALLED, PCB:Hole3_5_out6mm, symbol pcb_details:HOLE_METALLED
- added D6: PMEG2020, Diodes:SOD323, symbol Tittar_kl:D_Shottky
- D1: footprint (none) -> LEDs:LED_0603
- R22: value 1M -> 10k
- XL45: symbol Connectors_kl:USB_MICRO_2H -> Connectors_kl:USB_B
Connections:
- net +5v: now also D6.C
- net 5V_USB: now also R22.1, D6.A
- net GND: no longer XL45.5 (UGND)
- net RS485_INT_MCU_RX: no longer DA4.4 (TX), DD3.33 (ADC12-13/TX3/PC4), TP12.1
- new net RS485_INT_MCU_TX: DA4.4 (TX), DD3.33 (ADC12-13/TX3/PC4), TP12.1
- no-connect marks 32 -> 34
Other:
- moved on the sheet: L2, U1

Commit message: + Gerbers ready
Parts:
- C12, C18, C20, C23, C25, C26, C29, C30, C6: footprint Capacitors:CAP_0603 -> Capacitors:CAP_0603_Silks
Changed lines of the file:
@@
 F 0 "C29" V 19850 7600 50  0000 L CNN
 F 1 "0.1u" V 19850 7300 50  0000 L CNN
-F 2 "Capacitors:CAP_0603" H 19750 7500 60  0001 C CNN
+F 2 "Capacitors:CAP_0603_Silks" H 19750 7500 60  0001 C CNN
 F 3 "" H 19750 7500 60  0001 C CNN
 	1    19750 7500
@@
 F 0 "C30" V 19850 7900 50  0000 L CNN
 F 1 "0.1u" V 19850 7600 50  0000 L CNN
-F 2 "Capacitors:CAP_0603" H 19750 7800 60  0001 C CNN
+F 2 "Capacitors:CAP_0603_Silks" H 19750 7800 60  0001 C CNN
 F 3 "" H 19750 7800 60  0001 C CNN
 	1    19750 7800
@@
 F 0 "C25" V 18100 7800 50  0000 L CNN
 F 1 "0.1u" V 18100 7500 50  0000 L CNN
-F 2 "Capacitors:CAP_0603" H 18000 7700 60  0001 C CNN
+F 2 "Capacitors:CAP_0603_Silks" H 18000 7700 60  0001 C CNN
 F 3 "" H 18000 7700 60  0001 C CNN
 	1    18000 7700
@@
 F 0 "C26" H 19600 7150 50  0000 L CNN
 F 1 "0.1u" H 19600 6950 50  0000 L CNN
-F 2 "Capacitors:CAP_0603" H 19550 7050 60  0001 C CNN
+F 2 "Capacitors:CAP_0603_Silks" H 19550 7050 60  0001 C CNN
 F 3 "" H 19550 7050 60  0001 C CNN
 	1    19550 7050
@@
 F 0 "C6" H 3550 11700 50  0000 L CNN
 F 1 "0.1u" H 3550 11900 50  0000 L CNN
-F 2 "Capacitors:CAP_0603" V 3750 11650 28  0001 C BNN
+F 2 "Capacitors:CAP_0603_Silks" V 3750 11650 28  0001 C BNN
 F 3 "" H 3650 11800 60  0001 C CNN
 	1    3650 11800
@@
 F 0 "C12" H 6050 11750 50  0000 L CNN
 F 1 "0.1u" H 6050 11950 50  0000 L CNN
-F 2 "Capacitors:CAP_0603" V 6250 11700 28  0001 C BNN
+F 2 "Capacitors:CAP_0603_Silks" V 6250 11700 28  0001 C BNN
 F 3 "" H 6050 11750 60  0001 C CNN
 F 4 "0.5" H 6150 11850 60  0001 C CNN "Price"
@@
 F 0 "C18" H 8300 11750 50  0000 L CNN
 F 1 "0.1u" H 8300 11950 50  0000 L CNN
-F 2 "Capacitors:CAP_0603" V 8500 11700 28  0001 C BNN
+F 2 "Capacitors:CAP_0603_Silks" V 8500 11700 28  0001 C BNN
 F 3 "" H 8300 11750 60  0001 C CNN
 F 4 "0.5" H 8400 11850 60  0001 C CNN "Price"
@@
 F 0 "C20" H 10800 11750 50  0000 L CNN
 F 1 "0.1u" H 10800 11950 50  0000 L CNN
-F 2 "Capacitors:CAP_0603" V 11000 11700 28  0001 C BNN
+F 2 "Capacitors:CAP_0603_Silks" V 11000 11700 28  0001 C BNN
 F 3 "" H 10800 11750 60  0001 C CNN
 F 4 "0.5" H 10900 11850 60  0001 C CNN "Price"
@@
 F 0 "C23" H 13550 12100 50  0000 L CNN
 F 1 "0.1u" H 13550 12300 50  0000 L CNN
-F 2 "Capacitors:CAP_0603" V 13750 12050 28  0001 C BNN
+F 2 "Capacitors:CAP_0603_Silks" V 13750 12050 28  0001 C BNN
 F 3 "" H 13550 12100 60  0001 C CNN
 F 4 "0.5" H 13650 12200 60  0001 C CNN "Price"
@@
 	-1   0    0    -1
 $EndComp
-$Comp
-L Connectors_kl:CONN_GOST_1 XL22
-U 1 1 5DDD9D37
-P 3700 4250
-F 0 "XL22" H 3778 4240 40  0000 L CNN
-F 1 "CONN_GOST_1" H 3778 4203 40  0001 L CNN
-F 2 "PCB:Oval3x1.5" H 3850 4250 60  0001 C CNN
-F 3 "" H 3850 4250 60  0000 C CNN
-	1    3700 4250
-	-1   0    0    -1
-$EndComp
-$Comp
-L Connectors_kl:CONN_GOST_1 XL19
-U 1 1 5DDD9D45
-P 3700 3950
-F 0 "XL19" H 3778 3940 40  0000 L CNN
-F 1 "CONN_GOST_1" H 3778 3903 40  0001 L CNN
-F 2 "PCB:Oval3x1.5" H 3850 3950 60  0001 C CNN
-F 3 "" H 3850 3950 60  0000 C CNN
-	1    3700 3950
-	-1   0    0    -1
-$EndComp
 Wire Wire Line
 	3850 2950 4300 2950
@@
 F 3 "" H 8850 5150 60  0000 C CNN
 	1    8700 5150
-	1    0    0    -1
-$EndComp
-$Comp
-L Connectors_kl:CONN_GOST_1 XL29
-U 1 1 5DDEDD5F
-P 8700 5450
-F 0 "XL29" H 8778 5440 40  0000 L CNN
-F 1 "CONN_GOST_1" H 8778 5403 40  0001 L CNN
-F 2 "PCB:Oval3x1.5" H 8850 5450 60  0001 C CNN
-F 3 "" H 8850 5450 60  0000 C CNN
-	1    8700 5450
 	1    0    0    -1
 $EndComp
@@
 Wire Wire Line
 	21250 12200 21250 12450
+$Comp
+L Connectors_kl:CONN_GOST_1 XL19
+U 1 1 5DDD9D45
+P 3700 3950
+F 0 "XL19" H 3778 3940 40  0000 L CNN
+F 1 "CONN_GOST_1" H 3778 3903 40  0001 L CNN
+F 2 "PCB:Oval3x1.5" H 3850 3950 60  0001 C CNN
+F 3 "" H 3850 3950 60  0000 C CNN
+	1    3700 3950
+	-1   0    0    -1
+$EndComp
+$Comp
+L Connectors_kl:CONN_GOST_1 XL22
+U 1 1 5DDD9D37
+P 3700 4250
+F 0 "XL22" H 3778 4240 40  0000 L CNN
+F 1 "CONN_GOST_1" H 3778 4203 40  0001 L CNN
+F 2 "PCB:Oval3x1.5" H 3850 4250 60  0001 C CNN
+F 3 "" H 3850 4250 60  0000 C CNN
+	1    3700 4250
+	-1   0    0    -1
+$EndComp
+$Comp
+L Connectors_kl:CONN_GOST_1 XL29
+U 1 1 5DDEDD5F
+P 8700 5450
+F 0 "XL29" H 8778 5440 40  0000 L CNN
+F 1 "CONN_GOST_1" H 8778 5403 40  0001 L CNN
+F 2 "PCB:Oval3x1.5" H 8850 5450 60  0001 C CNN
+F 3 "" H 8850 5450 60  0000 C CNN
+	1    8700 5450
+	1    0    0    -1
+$EndComp
 $EndSCHEMATC

Commit message: + TControl
Parts:
- added D?: PMEG2020, Diodes:SOD323, symbol Tittar_kl:D_Shottky
Connections:
- net +5v: now also D?.A, D?.C
Other:
- note added: "Add Diode somehow"
