File: CtrlTree_hw/CtrlTree.kicad_pcb (KiCad board)
At the start: 4 copper layers, 71 x 40 mm, 146 parts, among them Q1 IRLML6401, Q2 IRLML0030, U1 USBLC6

Commit message: + Gerbers ready
Parts:
- C12, C18, C20, C23, C25, C26, C29, C30, C6: footprint Capacitors:CAP_0603 -> Capacitors:CAP_0603_Silks
- moved TP17 103.5 mm to (171.7, 85.0)
- moved D2 97.0 mm to (173.3, 80.1), turned to 90 degrees
- moved TP8 90.9 mm to (161.3, 80.7)
- moved TP1 90.5 mm to (141.6, 82.3)
- moved TP6 90.2 mm to (122.4, 79.6), turned to 90 degrees
- moved R2 88.7 mm to (139.3, 80.7)
- moved TP2 88.3 mm to (141.6, 80.7)
- moved XL49 87.9 mm to (134.2, 79.3), turned to -90 degrees
- moved D4 87.3 mm to (173.3, 85.1), turned to -90 degrees
- moved DA5 87.2 mm to (171.2, 110.1), turned to -90 degrees
- moved TP5 86.9 mm to (115.5, 78.8)
- moved R5 86.0 mm to (167.9, 90.0), turned to -90 degrees
- moved R11 85.9 mm to (171.7, 82.6), turned to -90 degrees
- moved Q2 84.6 mm to (119.9, 79.6), turned to 90 degrees
- moved XL46 84.5 mm to (179.1, 83.8), turned to 180 degrees
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Routing:
- net +5v: track 0.00 -> 1689.8 mm, vias 0 -> 20
- net GND: track 0.00 -> 377.7 mm, vias 0 -> 42
- net /SNS_PWR: track 0.00 -> 109.6 mm, vias 0 -> 4
- net PwrMCU: track 0.00 -> 103.8 mm, vias 0 -> 6
- net /SCL: track 0.00 -> 95.2 mm, vias 0 -> 6
- net +3v3: track 0.00 -> 93.8 mm, vias 0 -> 5
- net /SDA: track 0.00 -> 92.3 mm, vias 0 -> 6
- net /HEATER_CTRL: track 0.00 -> 57.0 mm, vias 0 -> 2
- net /SPI2_CS: track 0.00 -> 48.1 mm, vias 0 -> 2
- net /SPI2_MOSI: track 0.00 -> 47.9 mm, vias 0 -> 2
- net /SPI2_MISO: track 0.00 -> 47.4 mm, vias 0 -> 2
- net /SPI2_SCK: track 0.00 -> 47.3 mm, vias 0 -> 2
- net /b18: track 0.00 -> 47.1 mm, vias 0 -> 2
- net /b19: track 0.00 -> 43.0 mm, vias 0 -> 2
- net /SPI1_CS: track 0.00 -> 42.0 mm, vias 0 -> 2
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- added copper zone on B.Cu, net +5v
- added copper zone on F.Cu, net +5v
- added copper zone on In1.Cu, net +5v
- added copper zone on In2.Cu, net +5v
- added copper zone on F.Cu, net /PWR_IN
- added copper zone on B.Cu, net GND
- added copper zone on F.Cu, net GND
- added copper zone on In1.Cu, net GND
- added copper zone on In2.Cu, net GND
Other:
- net class Default: clearance 0.18 -> 0.15; trace_width 0.18 -> 0.15; via_dia 0.7 -> 0.6
- net class Wide: clearance 0.2 -> 0.22; via_dia 0.7 -> 0.6
- rule trace_clearance: 0.18 -> 0.15
- board text added: "+"
- board text added: "A"
- board text added: "B"
- board text added: "B0"
- board text added: "B1"
- board text added: "B10"
- board text added: "B11"
- board text added: "B12"
- board text added: "B13"
- board text added: "B14"
- board text added: "B15"
- board text added: "B16"
- board text added: "B17"
- board text added: "B18"
- board text added: "B19"
- board text added: "B2"
- board text added: "B20"
- board text added: "B21"
- board text added: "B22"
- board text added: "B23"
- board text added: "B24"
- board text added: "B25"
- board text added: "B26"
- board text added: "B3"
- board text added: "B4"
- board text added: "B5"
- board text added: "B6"
- board text added: "B7"
- board text added: "B8"
- board text added: "B9"
- board text added: "CS1"
- board text added: "CS2"
- board text added: "ControlTree v191231"
- board text added: "EE"
- board text added: "GND"
- board text added: "LED"
- board text added: "MISO1"
- board text added: "MISO2"
- board text added: "MOSI1"
- board text added: "MOSI2"
- board text added: "PWR 3v3"
- board text added: "RS232"
- board text added: "RS485 ext"
- board text added: "RS486 int"
- board text added: "SCK1"
- board text added: "SCK2"
- board text added: "Termo1"
- board text added: "Termo2"
- board text added: "Termo3"
- board text added: "USB"
- board text added: "rx"
- board text added: "tx"

Commit message: + saveregs * RReply
Parts:
- added D7: PMEG2020, Diodes:SOD323, F.Cu at (122.4, 80.9)
Other:
- net class Default removed
- net class Wide removed
