File: CtrlTree_hw/CtrlTree.kicad_sch (KiCad schematic)
At the start: 147 parts, among them Q1 IRLML6401, Q2 IRLML0030, U1 USBLC6

Commit message: + saveregs * RReply
Parts:
- gave numbers to parts that had none: 1
